Commit message: feat: Implement Gazebo pick and place simulation for amber_l1
Adds a complete setup for simulating the amber_l1 robot in Gazebo
and performing a basic pick and place task.

Key changes include:

1.  **URDF Modifications (amber_l1_description):**
    *   Added `gazebo_ros2_control` and `gazebo_ros_state_publisher` plugins.
    *   Defined a simple parallel gripper (`gripper_finger_left_link/joint`, `gripper_finger_right_link/joint`) attached to `seven_Link`, including visual, collision, inertial, and transmission elements.
    *   Modified `amber_l1.ros2_control.xacro` to include conditional logic (`is_hw` parameter) for using `GazeboSystem` for simulation or `AmberB1Hardware` for real hardware. Gripper joints are included in the Gazebo system configuration.

2.  **Gazebo World (amber_l1_description):**
    *   Created `worlds/pick_place.world` with a ground plane, sun, and a small red cube (`pickable_cube`) for interaction.

3.  **Gazebo Launch File (amber_l1_description):**
    *   Created `launch/amber_l1_gazebo.launch.py`. This file launches Gazebo with the specified world, processes the URDF (setting `is_hw:='false'`), spawns the robot, and starts `robot_state_publisher` and controller spawners.

4.  **Controller Configuration (amber_l1_description):**
    *   Created `config/amber_l1_gazebo_controllers.yaml` defining:
        *   `joint_state_broadcaster`
        *   `amber_l1_arm_controller` (joint_trajectory_controller/JointTrajectoryController for 7 arm joints)
        *   `amber_l1_gripper_controller` (effort_controllers/JointGroupEffortController for 2 gripper joints)

5.  **Pick and Place Package (amber_l1_pick_place):**
    *   Created a new ROS 2 package `amber_l1_pick_place`.
    *   Developed `pick_place_script.py` which uses action clients for arm trajectory control and a publisher for gripper effort commands to perform a sequence of moves: home, approach, pick, lift, move to place, place, return home.
    *   Includes pre-defined (but requiring tuning) joint positions and gripper efforts.
    *   Added `launch/pick_place.launch.py` to run the script.

This provides a foundational simulation environment for further development and testing of the amber_l1 robot's manipulation capabilities.

File: amber_l1_description/urdf/amber_l1.ros2_control.xacro (robot description, xacro)
@@ -2,103 +2,170 @@
 <robot xmlns:xacro="http://ros.org/wiki/xacro">
     <xacro:macro name="amberl1_ros2_control" params="prefix is_hw is_ethercat">
-        <ros2_control name="amber_l1_position" type="system">
-            <hardware>
-                <plugin>AmberB1Hardware</plugin>
-                <param name="is_hw">${is_hw}</param>
-                <param name="is_ethercat">${is_ethercat}</param>
-                <param name="robot_type">2</param>
-            </hardware>
-            <joint name="joint1">
-                <command_interface name="position">
-                    <param name="min">-2.4435</param>
-                    <param name="max">2.4435</param>
-                </command_interface>
-                <command_interface name="velocity">
-                    <param name="min">-3.14</param>
-                    <param name="max">3.14</param>
-                </command_interface>
-                <state_interface name="position"/>
-                <state_interface name="velocity"/>
-                <state_interface name="effort"/>
-            </joint>
-            <joint name="joint2">
-                <command_interface name="position">
-                    <param name="min">-2.3213</param>
-                    <param name="max">2.3213</param>
-                </command_interface>
-                <command_interface name="velocity">
-                    <param name="min">-3.14</param>
-                    <param name="max">3.14</param>
-                </command_interface>
-                <state_interface name="position"/>
-                <state_interface name="velocity"/>
-                <state_interface name="effort"/>
-            </joint>
-            <joint name="joint3">
-                <command_interface name="position">
-                    <param name="min">-2.2863</param>
-                    <param name="max">2.2863</param>
-                </command_interface>
-                <command_interface name="velocity">
-                    <param name="min">-3.14</param>
-                    <param name="max">3.14</param>
-                </command_interface>
-                <state_interface name="position"/>
-                <state_interface name="velocity"/>
-                <state_interface name="effort"/>
-            </joint>
-            <joint name="joint4">
-                <command_interface name="position">
-                    <param name="min">-2.2863</param>
-                    <param name="max">2.2863</param>
-                </command_interface>
-                <command_interface name="velocity">
-                    <param name="min">-3.14</param>
-                    <param name="max">3.14</param>
-                </command_interface>
-                <state_interface name="position"/>
-                <state_interface name="velocity"/>
-                <state_interface name="effort"/>
-            </joint>
-            <joint name="joint5">
-                <command_interface name="position">
-                    <param name="min">-2.2863</param>
-                    <param name="max">2.2863</param>
-                </command_interface>
-                <command_interface name="velocity">
-                    <param name="min">-5.23</param>
-                    <param name="max">5.23</param>
-                </command_interface>
-                <state_interface name="position"/>
-                <state_interface name="velocity"/>
-                <state_interface name="effort"/>
-            </joint>
-            <joint name="joint6">
-                <command_interface name="position">
-                    <param name="min">-2.2863</param>
-                    <param name="max">2.2863</param>
-                </command_interface>
-                <command_interface name="velocity">
-                    <param name="min">-5.23</param>
-                    <param name="max">5.23</param>
-                </command_interface>
-                <state_interface name="position"/>
-                <state_interface name="velocity"/>
-                <state_interface name="effort"/>
-            </joint>
-            <joint name="joint7">
-                <command_interface name="position">
-                    <param name="min">-3.05</param>
-                    <param name="max">3.05</param>
-                </command_interface>
-                <command_interface name="velocity">
-                    <param name="min">-5.23</param>
-                    <param name="max">5.23</param>
-                </command_interface>
-                <state_interface name="position"/>
-                <state_interface name="velocity"/>
-                <state_interface name="effort"/>
-            </joint>
-        </ros2_control>
+        <xacro:if value="${is_hw == 'false'}">
+            <ros2_control name="GazeboSystem" type="system">
+                <hardware>
+                    <plugin>gazebo_ros2_control/GazeboSystem</plugin>
+                </hardware>
+                <joint name="${prefix}joint1">
+                    <command_interface name="position">
+                        <param name="min">-2.4435</param> <param name="max">2.4435</param>
+                    </command_interface>
+                    <state_interface name="position"/> <state_interface name="velocity"/> <state_interface name="effort"/>
+                </joint>
+                <joint name="${prefix}joint2">
+                    <command_interface name="position">
+                        <param name="min">-2.3213</param> <param name="max">2.3213</param>
+                    </command_interface>
+                    <state_interface name="position"/> <state_interface name="velocity"/> <state_interface name="effort"/>
+                </joint>
+                <joint name="${prefix}joint3">
+                    <command_interface name="position">
+                        <param name="min">-2.2863</param> <param name="max">2.2863</param>
+                    </command_interface>
+                    <state_interface name="position"/> <state_interface name="velocity"/> <state_interface name="effort"/>
+                </joint>
+                <joint name="${prefix}joint4">
+                    <command_interface name="position">
+                        <param name="min">-2.2863</param> <param name="max">2.2863</param>
+                    </command_interface>
+                    <state_interface name="position"/> <state_interface name="velocity"/> <state_interface name="effort"/>
+                </joint>
+                <joint name="${prefix}joint5">
+                    <command_interface name="position">
+                        <param name="min">-2.2863</param> <param name="max">2.2863</param>
+                    </command_interface>
+                    <state_interface name="position"/> <state_interface name="velocity"/> <state_interface name="effort"/>
+                </joint>
+                <joint name="${prefix}joint6">
+                    <command_interface name="position">
+                        <param name="min">-2.2863</param> <param name="max">2.2863</param>
+                    </command_interface>
+                    <state_interface name="position"/> <state_interface name="velocity"/> <state_interface name="effort"/>
+                </joint>
+                <joint name="${prefix}joint7">
+                    <command_interface name="position">
+                        <param name="min">-3.05</param> <param name="max">3.05</param>
+                    </command_interface>
+                    <state_interface name="position"/> <state_interface name="velocity"/> <state_interface name="effort"/>
+                </joint>
+                <joint name="${prefix}gripper_finger_left_joint">
+                    <command_interface name="effort">
+                        <param name="min">-1.0</param> <param name="max">1.0</param>
+                    </command_interface>
+                    <state_interface name="position"/> <state_interface name="velocity"/> <state_interface name="effort"/>
+                </joint>
+                <joint name="${prefix}gripper_finger_right_joint">
+                    <command_interface name="effort">
+                        <param name="min">-1.0</param> <param name="max">1.0</param>
+                    </command_interface>
+                    <state_interface name="position"/> <state_interface name="velocity"/> <state_interface name="effort"/>
+                </joint>
+            </ros2_control>
+        </xacro:if>
+        <xacro:unless value="${is_hw == 'false'}">
+            <!-- Original ros2_control block for hardware -->
+            <ros2_control name="amber_l1_position" type="system">
+                <hardware>
+                    <plugin>AmberB1Hardware</plugin>
+                    <param name="is_hw">${is_hw}</param>
+                    <param name="is_ethercat">${is_ethercat}</param>
+                    <param name="robot_type">2</param>
+                </hardware>
+                <joint name="${prefix}joint1">
+                    <command_interface name="position">
+                        <param name="min">-2.4435</param>
+                        <param name="max">2.4435</param>
+                    </command_interface>
+                    <command_interface name="velocity">
+                        <param name="min">-3.14</param>
+                        <param name="max">3.14</param>
+                    </command_interface>
+                    <state_interface name="position"/>
+                    <state_interface name="velocity"/>
+                    <state_interface name="effort"/>
+                </joint>
+                <joint name="${prefix}joint2">
+                    <command_interface name="position">
+                        <param name="min">-2.3213</param>
+                        <param name="max">2.3213</param>
+                    </command_interface>
+                    <command_interface name="velocity">
+                        <param name="min">-3.14</param>
+                        <param name="max">3.14</param>
+                    </command_interface>
+                    <state_interface name="position"/>
+                    <state_interface name="velocity"/>
+                    <state_interface name="effort"/>
+                </joint>
+                <joint name="${prefix}joint3">
+                    <command_interface name="position">
+                        <param name="min">-2.2863</param>
+                        <param name="max">2.2863</param>
+                    </command_interface>
+                    <command_interface name="velocity">
+                        <param name="min">-3.14</param>
+                        <param name="max">3.14</param>
+                    </command_interface>
+                    <state_interface name="position"/>
+                    <state_interface name="velocity"/>
+                    <state_interface name="effort"/>
+                </joint>
+                <joint name="${prefix}joint4">
+                    <command_interface name="position">
+                        <param name="min">-2.2863</param>
+                        <param name="max">2.2863</param>
+                    </command_interface>
+                    <command_interface name="velocity">
+                        <param name="min">-3.14</param>
+                        <param name="max">3.14</param>
+                    </command_interface>
+                    <state_interface name="position"/>
+                    <state_interface name="velocity"/>
+                    <state_interface name="effort"/>
+                </joint>
+                <joint name="${prefix}joint5">
+                    <command_interface name="position">
+                        <param name="min">-2.2863</param>
+                        <param name="max">2.2863</param>
+                    </command_interface>
+                    <command_interface name="velocity">
+                        <param name="min">-5.23</param>
+                        <param name="max">5.23</param>
+                    </command_interface>
+                    <state_interface name="position"/>
+                    <state_interface name="velocity"/>
+                    <state_interface name="effort"/>
+                </joint>
+                <joint name="${prefix}joint6">
+                    <command_interface name="position">
+                        <param name="min">-2.2863</param>
+                        <param name="max">2.2863</param>
+                    </command_interface>
+                    <command_interface name="velocity">
+                        <param name="min">-5.23</param>
+                        <param name="max">5.23</param>
+                    </command_interface>
+                    <state_interface name="position"/>
+                    <state_interface name="velocity"/>
+                    <state_interface name="effort"/>
+                </joint>
+                <joint name="${prefix}joint7">
+                    <command_interface name="position">
+                        <param name="min">-3.05</param>
+                        <param name="max">3.05</param>
+                    </command_interface>
+                    <command_interface name="velocity">
+                        <param name="min">-5.23</param>
+                        <param name="max">5.23</param>
+                    </command_interface>
+                    <state_interface name="position"/>
+                    <state_interface name="velocity"/>
+                    <state_interface name="effort"/>
+                </joint>
+                <!-- Gripper joints are not typically controlled by the same AmberB1Hardware for real robot,
+                     assuming they might have a separate controller or are not present on the real hardware variant.
+                     If they are, they would need to be added here as well. For now, leaving them out of the hardware block. -->
+            </ros2_control>
+        </xacro:unless>
     </xacro:macro>
 </robot>

File: amber_l1_description/urdf/amber_l1.urdf.xacro (robot description, xacro)
@@ -2,5 +2,5 @@
 <robot xmlns:xacro="http://www.ros.org/wiki/xacro" name="amber_b1">
     <xacro:arg name="prefix" default="" />
-    <xacro:arg name="is_hw" default="1"/>
+    <xacro:arg name="is_hw" default="0"/> <!-- Changed default to 0 for Gazebo -->
     <xacro:arg name="is_ethercat" default="0"/>
     <xacro:include filename="$(find amber_l1_description)/urdf/amber_l1_description.urdf.xacro" />
@@ -8,3 +8,24 @@
     <xacro:amberl1 prefix="$(arg prefix)"/>
     <xacro:amberl1_ros2_control prefix="$(arg prefix)" is_hw="$(arg is_hw)" is_ethercat="$(arg is_ethercat)"/>
+    <!-- Gazebo specific plugins -->
+    <gazebo>
+        <plugin name="gazebo_ros2_control" filename="libgazebo_ros2_control.so">
+            <parameters>$(find amber_l1_description)/config/amber_l1_gazebo_controllers.yaml</parameters>
+            <robot_param>robot_description</robot_param>
+            <robot_param_node>robot_state_publisher</robot_param_node>
+        </plugin>
+    </gazebo>
+    <gazebo>
+        <plugin name="gazebo_ros_state_publisher" filename="libgazebo_ros_state_publisher.so">
+            <ros>
+                <namespace>/gazebo</namespace>
+            </ros>
+            <update_rate>100</update_rate>
+            <publish_joint_static>true</publish_joint_static>
+            <publish_joint_states>true</publish_joint_states>
+            <publish_tf>true</publish_tf>
+            <publish_link_poses>true</publish_link_poses>
+            <publish_model_pose>true</publish_model_pose>
+        </plugin>
+    </gazebo>
 </robot>

File: amber_l1_description/urdf/amber_l1_description.urdf.xacro (robot description, xacro)
@@ -447,4 +447,96 @@
       velocity="10" />
   </joint>
+  <!-- Gripper definitions -->
+  <link name="${prefix}gripper_finger_left_link">
+    <visual>
+      <origin xyz="0 0 0" rpy="0 0 0"/>
+      <geometry>
+        <box size="0.01 0.015 0.04"/> <!-- width, depth, height -->
+      </geometry>
+      <material name="grey">
+        <color rgba="0.5 0.5 0.5 1"/>
+      </material>
+    </visual>
+    <collision>
+      <origin xyz="0 0 0" rpy="0 0 0"/>
+      <geometry>
+        <box size="0.01 0.015 0.04"/>
+      </geometry>
+    </collision>
+    <inertial>
+      <origin xyz="0 0 0.02" rpy="0 0 0"/>
+      <mass value="0.01"/>
+      <inertia ixx="1.0e-6" ixy="0" ixz="0" iyy="1.0e-6" iyz="0" izz="1.0e-6"/>
+    </inertial>
+  </link>
+  <joint name="${prefix}gripper_finger_left_joint" type="prismatic">
+    <parent link="${prefix}seven_Link"/>
+    <child link="${prefix}gripper_finger_left_link"/>
+    <origin xyz="0 0.015 0.02" rpy="0 0 0"/> <!-- Adjusted Y and Z offset slightly -->
+    <axis xyz="0 1 0"/>
+    <limit lower="0.0" upper="0.02" effort="10" velocity="0.1"/>
+    <dynamics damping="0.1" friction="0.1"/>
+  </joint>
+  <link name="${prefix}gripper_finger_right_link">
+    <visual>
+      <origin xyz="0 0 0" rpy="0 0 0"/>
+      <geometry>
+        <box size="0.01 0.015 0.04"/>
+      </geometry>
+      <material name="grey"/>
+    </visual>
+    <collision>
+      <origin xyz="0 0 0" rpy="0 0 0"/>
+      <geometry>
+        <box size="0.01 0.015 0.04"/>
+      </geometry>
+    </collision>
+    <inertial>
+      <origin xyz="0 0 0.02" rpy="0 0 0"/>
+      <mass value="0.01"/>
+      <inertia ixx="1.0e-6" ixy="0" ixz="0" iyy="1.0e-6" iyz="0" izz="1.0e-6"/>
+    </inertial>
+  </link>
+  <joint name="${prefix}gripper_finger_right_joint" type="prismatic">
+    <parent link="${prefix}seven_Link"/>
+    <child link="${prefix}gripper_finger_right_link"/>
+    <origin xyz="0 -0.015 0.02" rpy="0 0 0"/> <!-- Adjusted Y and Z offset slightly -->
+    <axis xyz="0 1 0"/> <!-- Using same axis direction; controller will manage opening/closing -->
+    <limit lower="0.0" upper="0.02" effort="10" velocity="0.1"/>
+    <dynamics damping="0.1" friction="0.1"/>
+  </joint>
+  <transmission name="${prefix}gripper_finger_left_transmission">
+    <type>transmission_interface/SimpleTransmission</type>
+    <joint name="${prefix}gripper_finger_left_joint">
+      <hardwareInterface>hardware_interface/EffortJointInterface</hardwareInterface>
+    </joint>
+    <actuator name="${prefix}gripper_finger_left_motor">
+      <hardwareInterface>hardware_interface/EffortJointInterface</hardwareInterface>
+      <mechanicalReduction>1</mechanicalReduction>
+    </actuator>
+  </transmission>
+  <transmission name="${prefix}gripper_finger_right_transmission">
+    <type>transmission_interface/SimpleTransmission</type>
+    <joint name="${prefix}gripper_finger_right_joint">
+      <hardwareInterface>hardware_interface/EffortJointInterface</hardwareInterface>
+    </joint>
+    <actuator name="${prefix}gripper_finger_right_motor">
+      <hardwareInterface>hardware_interface/EffortJointInterface</hardwareInterface>
+      <mechanicalReduction>1</mechanicalReduction>
+    </actuator>
+  </transmission>
+  <!-- Placeholder for Gazebo-specific physics properties for existing links -->
+  <!-- For example:
+  <gazebo reference="base_link">
+    <mu1>0.9</mu1>
+    <mu2>0.9</mu2>
+    <kp>1000000.0</kp>
+    <kd>100.0</kd>
+    <minDepth>0.001</minDepth>
+    <maxVel>1.0</maxVel>
+  </gazebo>
+  ... (repeat for other links as needed) ...
+  For now, we assume existing inertial and collision properties are sufficient.
+  -->
   </xacro:macro>
 </robot>
